Commit message: feat: added RGB-D Camera

File: src/my_robot/urdf/my_robot.xacro (robot description, xacro)
@@ -187,3 +187,13 @@
     </visual>
   </link>
+<joint name="camera_optical_joint" type="fixed">
+    <origin xyz="0 0 0" rpy="-1.5707 0 -1.5707"/>
+    <parent link="camera_link"/>
+    <child link="camera_link_optical"/>
+  </joint>
+  <link name="camera_link_optical">
+  </link>
+  <gazebo reference="camera_link">
+    <material>Gazebo/Green</material>
+  </gazebo>
 </robot>

Commit message: feat: added mapping and localization launch files

File: src/my_robot/urdf/my_robot.xacro (robot description, xacro)
@@ -189,11 +189,8 @@
 <joint name="camera_optical_joint" type="fixed">
     <origin xyz="0 0 0" rpy="-1.5707 0 -1.5707"/>
-    <parent link="camera_link"/>
+    <parent link="camera"/>
     <child link="camera_link_optical"/>
   </joint>
   <link name="camera_link_optical">
   </link>
-  <gazebo reference="camera_link">
-    <material>Gazebo/Green</material>
-  </gazebo>
 </robot>
